Commit message: Added inertia tags to URDF of arm and hand

File: franka_description/robots/hand.xacro (robot description, xacro)
@@ -10,5 +10,15 @@
       </joint>
     </xacro:unless>
+    <xacro:arg name="gazebo" default="true"/>
+    <xacro:if value="$(arg gazebo)">
+      <!-- Gazebo Tags -->
+      <xacro:include filename="$(find franka_description)/robots/hand.gazebo.xacro"/>
+    </xacro:if>
     <link name="${ns}_hand">
+      <inertial>
+        <mass value="0.73" />
+        <origin xyz="0 0.0015244 0.0275912" rpy="0 0 0" />
+        <inertia ixx="0.00278560230025" ixy="0.0" ixz="0.0" iyy="0.000400033405336" iyz="0.0" izz="0.00256378041832" />
+      </inertial>
       <visual>
         <geometry>
@@ -54,4 +64,9 @@
     </link>
     <link name="${ns}_leftfinger">
+      <inertial>
+        <mass value="0.1" />
+        <origin xyz="0 0.0145644 0.0227941" rpy="0 0 0" />
+        <inertia ixx="3.01220925051e-05" ixy="0.0" ixz="0.0" iyy="2.95873808038e-05" iyz="0.0" izz="6.95125211657e-06" />
+      </inertial>
       <visual>
         <geometry>
@@ -61,4 +76,9 @@
     </link>
     <link name="${ns}_rightfinger">
+      <inertial>
+        <mass value="0.1" />
+        <origin xyz="0 0.0145644 0.0227941" rpy="0 0 ${pi}" />
+        <inertia ixx="3.01220925051e-05" ixy="0.0" ixz="0.0" iyy="2.95873808038e-05" iyz="0.0" izz="6.95125211657e-06" />
+      </inertial>
       <visual>
         <origin xyz="0 0 0" rpy="0 0 ${pi}"/>

File: franka_description/robots/panda_arm.xacro (robot description, xacro)
@@ -11,5 +11,15 @@
       </joint>
     </xacro:unless>
+    <xacro:arg name="gazebo" default="true"/>
+    <xacro:if value="$(arg gazebo)">
+      <!-- Gazebo Tags -->
+      <xacro:include filename="$(find franka_description)/robots/panda_arm.gazebo.xacro"/>
+    </xacro:if>
     <link name="${arm_id}_link0">
+      <inertial>
+        <mass value="2.92" />
+        <origin xyz="-0.025566 -2.88e-05 0.057332" rpy="0 0 0" />
+        <inertia ixx="0.00782229414331" ixy="-1.56191622996e-05" ixz="-0.00126005738123" iyy="0.0109027971813" iyz="1.08233858202e-05" izz="0.0102355503949" />
+      </inertial>
       <visual>
         <geometry>
@@ -37,4 +47,9 @@
     </link>
     <link name="${arm_id}_link1">
+      <inertial>
+        <mass value="2.74" />
+        <origin xyz="0 -0.0324958 -0.0675818" rpy="0 0 0" />
+        <inertia ixx="0.0180416958283" ixy="0.0" ixz="0.0" iyy="0.0159136071891" iyz="0.0046758424612" izz="0.00620690827127" />
+      </inertial>
       <visual>
         <geometry>
@@ -70,4 +85,9 @@
     </joint>
     <link name="${arm_id}_link2">
+      <inertial>
+        <mass value="2.74" />
+        <origin xyz="0 -0.06861 0.0322285" rpy="0 0 0" />
+        <inertia ixx="0.0182856182281" ixy="0.0" ixz="0.0" iyy="0.00621358421175" iyz="-0.00472844221905" izz="0.0161514346309" />
+      </inertial>
       <visual>
         <geometry>
@@ -103,4 +123,9 @@
     </joint>
     <link name="${arm_id}_link3">
+      <inertial>
+        <mass value="2.38" />
+        <origin xyz="0.0469893 0.0316374 -0.031704" rpy="0 0 0" />
+        <inertia ixx="0.00771376630908" ixy="-0.00248490625138" ixz="-0.00332147581033" iyy="0.00989108008727" iyz="-0.00217796151484" izz="0.00811723558464" />
+      </inertial>
       <visual>
         <geometry>
@@ -136,4 +161,9 @@
     </joint>
     <link name="${arm_id}_link4">
+      <inertial>
+        <mass value="2.38" />
+        <origin xyz="-0.0360446 0.0336853 0.031882" rpy="0 0 0" />
+        <inertia ixx="0.00799663881132" ixy="0.00347095570217" ixz="-0.00241222942995" iyy="0.00825390705278" iyz="0.00235774044121" izz="0.0102515004345" />
+      </inertial>
       <visual>
         <geometry>
@@ -169,4 +199,9 @@
     </joint>
     <link name="${arm_id}_link5">
+      <inertial>
+        <mass value="2.74" />
+        <origin xyz="0 0.0610427 -0.104176" rpy="0 0 0" />
+        <inertia ixx="0.030371374513" ixy="6.50283587108e-07" ixz="-1.05129179916e-05" iyy="0.0288752887402" iyz="-0.00775653445787" izz="0.00444134056164" />
+      </inertial>
       <visual>
         <geometry>
@@ -220,4 +255,9 @@
     </joint>
     <link name="${arm_id}_link6">
+      <inertial>
+        <mass value="1.55" />
+        <origin xyz="0.0510509 0.009108 0.0106343" rpy="0 0 0" />
+        <inertia ixx="0.00303336450376" ixy="-0.000437276865508" ixz="0.000629257294877" iyy="0.00404479911567" iyz="0.000130472021025" izz="0.00558234286039" />
+      </inertial>
       <visual>
         <geometry>
@@ -253,4 +293,9 @@
     </joint>
     <link name="${arm_id}_link7">
+      <inertial>
+        <mass value="0.54" />
+        <origin xyz="0.0109695 0.0107965 0.0650411" rpy="0 0 0" />
+        <inertia ixx="0.000888868887021" ixy="-0.00012239074652" ixz="3.98699829666e-05" iyy="0.000888001373233" iyz="-9.33825115206e-05" izz="0.0007176834609" />
+      </inertial>
       <visual>
         <geometry>

Commit message: Changes to robot description to allow grasping in simulation

File: franka_description/robots/hand.xacro (robot description, xacro)
@@ -44,5 +44,5 @@
         </geometry>
       </collision>
-      <collision>
+      <!-- <collision>
         <origin xyz="0 0 0.1" rpy="0 ${pi/2} ${pi/2}"/>
         <geometry>
@@ -61,5 +61,5 @@
           <sphere radius="${0.02+safety_distance}"  />
         </geometry>
-      </collision>
+      </collision> -->
     </link>
     <link name="${ns}_leftfinger">
@@ -74,4 +74,9 @@
         </geometry>
       </visual>
+      <collision>
+        <geometry>
+          <mesh filename="package://franka_description/meshes/visual/finger.dae"/>
+        </geometry>
+      </collision>
     </link>
     <link name="${ns}_rightfinger">
@@ -87,4 +92,10 @@
         </geometry>
       </visual>
+      <collision>
+        <origin xyz="0 0 0" rpy="0 0 ${pi}"/>
+        <geometry>
+          <mesh filename="package://franka_description/meshes/visual/finger.dae"/>
+        </geometry>
+      </collision>
    </link>
     <joint name="${ns}_finger_joint1" type="prismatic">

File: franka_description/robots/panda_arm.xacro (robot description, xacro)
@@ -331,5 +331,5 @@
     </joint>
     <link name="${arm_id}_link8">
-      <collision>
+      <!-- <collision>
         <origin xyz="0.0424 0.0424 -0.0250" rpy="${pi} ${pi/2} ${pi/2}"/>
         <geometry>
@@ -348,5 +348,5 @@
           <sphere radius="${0.03+safety_distance}"  />
         </geometry>
-      </collision>
+      </collision> -->
     </link>
     <joint name="${arm_id}_joint8" type="fixed">
