Commit message: Changed inertia values to ones from another repo
https://github.com/erdalpekel/franka_ros.git

File: franka_description/robots/hand.xacro (robot description, xacro)
@@ -53,7 +53,7 @@
       </collision> -->
       <inertial>
-        <mass value="0.73" />
-        <origin xyz="0 0.0015244 0.0275912" rpy="0 0 0" />
-        <inertia ixx="0.00278560230025" ixy="0.0" ixz="0.0" iyy="0.000400033405336" iyz="0.0" izz="0.00256378041832" />
+        <origin xyz="0 0 0" rpy="0 0 0" />
+        <mass value="0.68" />
+        <inertia ixx="0.1" ixy="0.0" ixz="0.0" iyy="0.1" iyz="0.0" izz="0.1" />
       </inertial>
     </link>
@@ -70,7 +70,7 @@
       </collision>
       <inertial>
-        <mass value="0.1" />
-        <origin xyz="0 0.0145644 0.0227941" rpy="0 0 0" />
-        <inertia ixx="3.01220925051e-05" ixy="0.0" ixz="0.0" iyy="2.95873808038e-05" iyz="0.0" izz="6.95125211657e-06" />
+        <origin xyz="0 0 0" rpy="0 0 0" />
+        <mass value="0.68" />
+        <inertia ixx="0.1" ixy="0.0" ixz="0.0" iyy="0.1" iyz="0.0" izz="0.1" />
       </inertial>
     </link>
@@ -89,7 +89,7 @@
       </collision>
       <inertial>
-        <mass value="0.1" />
-        <origin xyz="0 0.0145644 0.0227941" rpy="0 0 ${pi}" />
-        <inertia ixx="3.01220925051e-05" ixy="0.0" ixz="0.0" iyy="2.95873808038e-05" iyz="0.0" izz="6.95125211657e-06" />
+        <origin xyz="0 0 0" rpy="0 0 0" />
+        <mass value="0.68" />
+        <inertia ixx="0.1" ixy="0.0" ixz="0.0" iyy="0.1" iyz="0.0" izz="0.1" />
       </inertial>
    </link>

File: franka_description/robots/panda_arm.xacro (robot description, xacro)
@@ -37,8 +37,8 @@
       </collision>
       <inertial>
-        <mass value="2.92" />
-        <origin xyz="-0.025566 -2.88e-05 0.057332" rpy="0 0 0" />
-        <inertia ixx="0.00782229414331" ixy="-1.56191622996e-05" ixz="-0.00126005738123" iyy="0.0109027971813" iyz="1.08233858202e-05" izz="0.0102355503949" />
-      </inertial>
+          <origin xyz="0 0 0" rpy="0 0 0" />
+          <mass value="3.06"/>
+          <inertia ixx="0.3" ixy="0.0" ixz="0.0" iyy="0.3" iyz="0.0" izz="0.3" />
+        </inertial>
     </link>
     <link name="${arm_id}_link1">
@@ -49,4 +49,9 @@
       </visual>
       <collision>
+        <geometry>
+          <mesh filename="package://${description_pkg}/meshes/collision/link1.stl"/>
+        </geometry>
+      </collision>
+      <!-- <collision>
         <origin xyz="0 0 -0.1915" rpy="0 0 0"/>
         <geometry>
@@ -65,10 +70,10 @@
           <sphere radius="${0.06+safety_distance}" />
         </geometry>
-      </collision>
-      <inertial>
-        <mass value="2.74" />
-        <origin xyz="0 -0.0324958 -0.0675818" rpy="0 0 0" />
-        <inertia ixx="0.0180416958283" ixy="0.0" ixz="0.0" iyy="0.0159136071891" iyz="0.0046758424612" izz="0.00620690827127" />
-      </inertial>
+      </collision> -->
+      <inertial>
+          <origin xyz="0 0 0" rpy="0 0 0" />
+          <mass value="2.34"/>
+          <inertia ixx="0.3" ixy="0.0" ixz="0.0" iyy="0.3" iyz="0.0" izz="0.3" />
+        </inertial>
     </link>
     <joint name="${arm_id}_joint1" type="revolute">
@@ -105,8 +110,8 @@
       </collision>
       <inertial>
-        <mass value="2.74" />
-        <origin xyz="0 -0.06861 0.0322285" rpy="0 0 0" />
-        <inertia ixx="0.0182856182281" ixy="0.0" ixz="0.0" iyy="0.00621358421175" iyz="-0.00472844221905" izz="0.0161514346309" />
-      </inertial>
+          <origin xyz="0 0 0" rpy="0 0 0" />
+          <mass value="2.36"/>
+          <inertia ixx="0.3" ixy="0.0" ixz="0.0" iyy="0.3" iyz="0.0" izz="0.3" />
+        </inertial>
     </link>
     <joint name="${arm_id}_joint2" type="revolute">
@@ -143,8 +148,8 @@
       </collision>
       <inertial>
-        <mass value="2.38" />
-        <origin xyz="0.0469893 0.0316374 -0.031704" rpy="0 0 0" />
-        <inertia ixx="0.00771376630908" ixy="-0.00248490625138" ixz="-0.00332147581033" iyy="0.00989108008727" iyz="-0.00217796151484" izz="0.00811723558464" />
-      </inertial>
+          <origin xyz="0 0 0" rpy="0 0 0" />
+          <mass value="2.38"/>
+          <inertia ixx="0.3" ixy="0.0" ixz="0.0" iyy="0.3" iyz="0.0" izz="0.3" />
+        </inertial>
     </link>
     <joint name="${arm_id}_joint3" type="revolute">
@@ -181,8 +186,8 @@
       </collision>
       <inertial>
-        <mass value="2.38" />
-        <origin xyz="-0.0360446 0.0336853 0.031882" rpy="0 0 0" />
-        <inertia ixx="0.00799663881132" ixy="0.00347095570217" ixz="-0.00241222942995" iyy="0.00825390705278" iyz="0.00235774044121" izz="0.0102515004345" />
-      </inertial>
+          <origin xyz="0 0 0" rpy="0 0 0" />
+          <mass value="2.43"/>
+          <inertia ixx="0.3" ixy="0.0" ixz="0.0" iyy="0.3" iyz="0.0" izz="0.3" />
+        </inertial>
     </link>
     <joint name="${arm_id}_joint4" type="revolute">
@@ -237,8 +242,8 @@
       </collision>
       <inertial>
-        <mass value="2.74" />
-        <origin xyz="0 0.0610427 -0.104176" rpy="0 0 0" />
-        <inertia ixx="0.030371374513" ixy="6.50283587108e-07" ixz="-1.05129179916e-05" iyy="0.0288752887402" iyz="-0.00775653445787" izz="0.00444134056164" />
-      </inertial>
+          <origin xyz="0 0 0" rpy="0 0 0" />
+          <mass value="3.5"/>
+          <inertia ixx="0.3" ixy="0.0" ixz="0.0" iyy="0.3" iyz="0.0" izz="0.3" />
+        </inertial>
     </link>
     <joint name="${arm_id}_joint5" type="revolute">
@@ -275,8 +280,8 @@
       </collision>
       <inertial>
-        <mass value="1.55" />
-        <origin xyz="0.0510509 0.009108 0.0106343" rpy="0 0 0" />
-        <inertia ixx="0.00303336450376" ixy="-0.000437276865508" ixz="0.000629257294877" iyy="0.00404479911567" iyz="0.000130472021025" izz="0.00558234286039" />
-      </inertial>
+          <origin xyz="0 0 0" rpy="0 0 0" />
+          <mass value="1.47"/>
+          <inertia ixx="0.3" ixy="0.0" ixz="0.0" iyy="0.3" iyz="0.0" izz="0.3" />
+        </inertial>
     </link>
     <joint name="${arm_id}_joint6" type="revolute">
@@ -313,8 +318,8 @@
       </collision>
       <inertial>
-        <mass value="0.54" />
-        <origin xyz="0.0109695 0.0107965 0.0650411" rpy="0 0 0" />
-        <inertia ixx="0.000888868887021" ixy="-0.00012239074652" ixz="3.98699829666e-05" iyy="0.000888001373233" iyz="-9.33825115206e-05" izz="0.0007176834609" />
-      </inertial>
+          <origin xyz="0 0 0" rpy="0 0 0" />
+          <mass value="0.45"/>
+          <inertia ixx="0.3" ixy="0.0" ixz="0.0" iyy="0.3" iyz="0.0" izz="0.3" />
+        </inertial>
     </link>
     <joint name="${arm_id}_joint7" type="revolute">
@@ -346,8 +351,8 @@
       </collision> -->
       <inertial>
-        <origin rpy="0 0 0" xyz="0 0 0"/>
-        <mass value="0.45"/>
-        <inertia ixx="0.3" ixy="0.0" ixz="0.0" iyy="0.3" iyz="0.0" izz="0.3"/>
-      </inertial>
+          <origin xyz="0 0 0" rpy="0 0 0" />
+          <mass value="0.45"/>
+          <inertia ixx="0.3" ixy="0.0" ixz="0.0" iyy="0.3" iyz="0.0" izz="0.3" />
+        </inertial>
     </link>
     <joint name="${arm_id}_joint8" type="fixed">
