Commit message: Avoid duplicate gazebo controllers

File: franka_description/robots/panda_arm.gazebo.xacro (robot description, xacro)
@@ -1,5 +1,5 @@
 <?xml version='1.0' encoding='utf-8'?>
 <robot xmlns:xacro="http://www.ros.org/wiki/xacro" name="panda">
-  <xacro:macro name="panda_gazebo" params="arm_id">
+  <xacro:macro name="panda_gazebo" params="arm_id include_gazebo_control:=true">
     <gazebo reference="${arm_id}_link0"/>
     <gazebo reference="${arm_id}_link1"/>
@@ -42,5 +42,6 @@
       </actuator>
     </transmission>
-    <transmission name="${arm_id}_finger_joint2_trans">
+    <!-- Don't need this since the second joint is to be mimicked -->
+    <!-- <transmission name="${arm_id}_finger_joint2_trans">
       <type>transmission_interface/SimpleTransmission</type>
       <joint name="${arm_id}_finger_joint2">
@@ -50,12 +51,14 @@
         <mechanicalReduction>1</mechanicalReduction>
       </actuator>
-    </transmission>
+    </transmission> -->
+    <xacro:if value="${include_gazebo_control}">
+      <gazebo>
+        <plugin name="gazebo_ros_control" filename="libgazebo_ros_control.so">
+          <robotNamespace>/</robotNamespace>
+        </plugin>
+      </gazebo>
+    </xacro:if>
+    <!-- gazebo plugin to mimic finger joints -->
     <gazebo>
-      <plugin name="gazebo_ros_control" filename="libgazebo_ros_control.so">
-        <robotNamespace>/</robotNamespace>
-      </plugin>
-    </gazebo>
-    <!-- gazebo plugin to mimic finger joints -->
-    <!-- <gazebo>
       <plugin name="panda_hand_mimic_joint_plugin" filename="libroboticsgroup_gazebo_mimic_joint_plugin.so">
         <joint>panda_finger_joint1</joint>
@@ -64,5 +67,5 @@
         <multiplier>2.0</multiplier>
       </plugin>
-    </gazebo> -->
+    </gazebo>
   </xacro:macro>
 </robot>
